File: PCB_Design/daughter_board/bms3_1.sch (EAGLE design)
At the start: 160 parts, among them T1 RTR020P02, T10 RTR020P02, T11 RTR020P02, T12 RTR020P02, T2 RTR020P02, T3 RTR020P02, T4 RTR020P02, T5 RTR020P02, T6 RTR020P02, T7 RTR020P02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

Commit message: more 0603
Parts:
- C1, C10, C11, C12, C13, C14, C15, C18, C19, C2, C20, C3, C6: device rcl:C-EUC0402 -> rcl:C-EUC0603
- R1, R13, R16, R17, R2, R20, R21, R25, R26, R3, R30, R31, R35, R36, R40, R41, R45, R46, R51, R60, R61, R65, R66, R70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: device rcl:R-US_R0402 -> rcl:R-US_R0603
